Commit message: Created Lidar

File: description/colours.xacro (robot description, xacro)
@@ -13,3 +13,6 @@
     <color rgba="0 0 0 1"/>
 </material>
+<material name="red">
+    <color rgba="1 0 0 1"/>
+</material>
 </robot>

File: description/robot.urdf.xacro (robot description, xacro)
@@ -5,3 +5,4 @@
     <xacro:include filename="colours.xacro" />
     <xacro:include filename="gazebo_control.xacro" />
+    <xacro:include filename="lidar.xacro" />
 </robot>

File: description/robot_core.xacro (robot description, xacro)
@@ -109,3 +109,6 @@
     <mu2 value="0.001"/>
 </gazebo>
+<gazebo reference="laser_frame">
+    <material>Gazebo/Red</material>
+</gazebo>
 </robot>
