Commit message: Created Gazebo control world

File: description/robot.urdf.xacro (robot description, xacro)
@@ -4,3 +4,4 @@
     <xacro:include filename="robot_core.xacro" />
     <xacro:include filename="colours.xacro" />
+    <xacro:include filename="gazebo_control.xacro" />
 </robot>

File: description/robot_core.xacro (robot description, xacro)
@@ -27,4 +27,7 @@
     </xacro:inertial_box>
 </link>
+<gazebo reference="chassis">
+    <material>Gazebo/White</material>
+</gazebo>
 <!-- LEFT WHEEL -->
 <joint name="left_wheel_joint" type="continuous">
@@ -50,4 +53,7 @@
     </xacro:inertial_cylinder>
 </link>
+   <gazebo reference="left_wheel">
+    <material>Gazebo/Blue</material>
+</gazebo>
 <!-- RIGHT WHEEL -->
 <joint name="right_wheel_joint" type="continuous">
@@ -73,4 +79,7 @@
     </xacro:inertial_cylinder>
 </link>
+<gazebo reference="right_wheel">
+    <material>Gazebo/Blue</material>
+</gazebo>
 <!-- CASTER WHEEL -->
 <joint name="caster_wheel_joint" type="fixed">
@@ -95,3 +104,8 @@
     </xacro:inertial_sphere>
 </link>
+ <gazebo reference="caster_wheel">
+    <material>Gazebo/Blue</material>
+    <mu1 value="0.001"/>
+    <mu2 value="0.001"/>
+</gazebo>
 </robot>

Commit message: Created camera

File: description/robot.urdf.xacro (robot description, xacro)
@@ -6,3 +6,4 @@
     <xacro:include filename="gazebo_control.xacro" />
     <xacro:include filename="lidar.xacro" />
+    <xacro:include filename="camera.xacro" />
 </robot>

File: description/robot_core.xacro (robot description, xacro)
@@ -112,3 +112,6 @@
     <material>Gazebo/Red</material>
 </gazebo>
+<gazebo reference="camera_link">
+    <material>Gazebo/Red</material>
+</gazebo>
 </robot>

Commit message: Solved problems

File: description/robot.urdf.xacro (robot description, xacro)
@@ -1,7 +1,14 @@
 <?xml version="1.0"?>
 <robot xmlns:xacro="http://www.ros.org/wiki/xacro"  name="robot">
+    <xacro:arg name="use_ros2_control" default="true"/>
     <!-- Example link -->
     <xacro:include filename="robot_core.xacro" />
+    <xacro:if value="$(arg use_ros2_control)">
     <xacro:include filename="ros2_control.xacro" />
+    </xacro:if>
+    <xacro:unless value="$(arg use_ros2_control)">
+        <xacro:include filename="gazebo_control.xacro" />
+    </xacro:unless>
+    <!--<xacro:include filename="ros2_control.xacro" /> -->
     <xacro:include filename="colours.xacro" />
    <!-- <xacro:include filename="gazebo_control.xacro" /> -->

File: description/robot_core.xacro (robot description, xacro)
@@ -40,5 +40,5 @@
     <visual>
         <geometry>
-            <cylinder length="0.04" radius="0.05" />/>
+            <cylinder length="0.04" radius="0.05" />
         </geometry>
         <material name="blue"/>
@@ -46,5 +46,5 @@
     <collision>
         <geometry>
-            <cylinder length="0.04" radius="0.05" />/>
+            <sphere radius="0.05" />
         </geometry>
     </collision>
@@ -66,5 +66,5 @@
     <visual>
         <geometry>
-            <cylinder length="0.04" radius="0.05" />/>
+            <cylinder length="0.04" radius="0.05" />
         </geometry>
         <material name="blue"/>
@@ -72,5 +72,5 @@
     <collision>
         <geometry>
-            <cylinder length="0.04" radius="0.05" />/>
+            <sphere radius="0.05"/>
         </geometry>
     </collision>
